Commit message: fixing the mesh directory zed_msgs to zed_description

File: zed_wrapper/urdf/zed_macro.urdf.xacro (robot description, xacro)
@@ -162,5 +162,5 @@
           <origin xyz="${screw_offset_x} 0 ${screw_offset_z}" rpy="0 0 0"/>
           <geometry>
-            <mesh filename="file://$(find zed_msgs)/meshes/${model}.stl"/>
+            <mesh filename="file://$(find zed_description)/meshes/${model}.stl"/>
           </geometry>
             <material name="zed_mat">
@@ -171,5 +171,5 @@
           <origin xyz="${screw_offset_x} 0 ${screw_offset_z}" rpy="0 0 0"/>
           <geometry>
-            <mesh filename="file://$(find zed_msgs)/meshes/${model}.stl"/>
+            <mesh filename="file://$(find zed_description)/meshes/${model}.stl"/>
           </geometry>
         </collision>
@@ -188,5 +188,5 @@
             <origin xyz="0 0 0" rpy="0 0 0"/>
             <geometry>
-              <mesh filename="file://$(find zed_msgs)/meshes/${model}.stl"/>
+              <mesh filename="file://$(find zed_description)/meshes/${model}.stl"/>
             </geometry>
             <material name="zed_mat">
@@ -197,5 +197,5 @@
             <origin xyz="0 0 0" rpy="0 0 0"/>
             <geometry>
-              <mesh filename="file://$(find zed_msgs)/meshes/${model}.stl"/>
+              <mesh filename="file://$(find zed_description)/meshes/${model}.stl"/>
             </geometry>
           </collision>
@@ -219,5 +219,5 @@
             <origin xyz="0 0 0" rpy="0 0 0"/>
             <geometry>
-              <mesh filename="file://$(find zed_msgs)/meshes/${model}.stl"/>
+              <mesh filename="file://$(find zed_description)/meshes/${model}.stl"/>
             </geometry>
             <material name="zed_mat">
@@ -228,5 +228,5 @@
             <origin xyz="0 0 0" rpy="0 0 0"/>
             <geometry>
-              <mesh filename="file://$(find zed_msgs)/meshes/${model}.stl"/>
+              <mesh filename="file://$(find zed_description)/meshes/${model}.stl"/>
             </geometry>
           </collision>
